File: hardware/side-board/side-board.kicad_sch (KiCad schematic)
At the start: 25 parts, among them IC101 TPS62933DRLR, IC102 NUP2105LT1G, J101 Inter-board Connector

Commit message: Segregated specific libs into shared libs
Parts:
- D101: footprint side-board:DIOM5436X244N -> vector:DIOM5436X244N; symbol side-board:SMBJ18A-E3_52 -> vector:SMBJ18A-E3_52
- IC101: footprint side-board:SOTFL50P160X60-8N -> vector:SOTFL50P160X60-8N; symbol side-board:TPS62933DRLR -> vector:TPS62933DRLR
- IC102: footprint side-board:SOT96P237X111-3N -> vector:SOT96P237X111-3N; symbol side-board:NUP2105LT1G -> vector:NUP2105LT1G
Changed lines of the file:
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@@
 	)
 	(symbol
-		(lib_id "side-board:SMBJ18A-E3_52")
+		(lib_id "vector:SMBJ18A-E3_52")
 		(at 127.635 156.21 270)
 		(unit 1)
@@
 			)
 		)
-		(property "Footprint" "side-board:DIOM5436X244N"
+		(property "Footprint" "vector:DIOM5436X244N"
 			(at 33.985 166.37 0)
 			(hide yes)
@@
 	)
 	(symbol
-		(lib_id "side-board:TPS62933DRLR")
+		(lib_id "vector:TPS62933DRLR")
 		(at 73.66 38.735 0)
 		(unit 1)
@@
 			)
 		)
-		(property "Footprint" "side-board:SOTFL50P160X60-8N"
+		(property "Footprint" "vector:SOTFL50P160X60-8N"
 			(at 95.25 133.655 0)
 			(hide yes)
@@
 	)
 	(symbol
-		(lib_id "side-board:NUP2105LT1G")
+		(lib_id "vector:NUP2105LT1G")
 		(at 46.99 153.035 270)
 		(unit 1)
@@
 			)
 		)
-		(property "Footprint" "side-board:SOT96P237X111-3N"
+		(property "Footprint" "vector:SOT96P237X111-3N"
 			(at -47.93 174.625 0)
 			(hide yes)
