File: hardware/carrier-cm5/cm5_highspeed.kicad_sch (KiCad schematic)
At the start: 35 parts, among them J20 CAM0, J21 CAM1, J9 USB3_A stacked, U20 AP2553W6, U21 AP2553W6, U22 TPD4EUSB30, U23 TPD4EUSB30

Commit message: Updated schematic on CM5 carrier
Parts:
- renumbered C9 to C201, C18 to C202, C13 to C203, C20 to C204, C70 to C205, C73 to C206, C71 to C207, C74 to C208, C72 to C209, C75 to C210, D3 to D201, D4 to D202, D5 to D203, J20 to J201, J21 to J202, J9 to J203, Module1 to Module201, R50 to R201, R51 to R202, R40 to R203, R41 to R204, R52 to R205, TP30 to TP201, TP33 to TP202, TP36 to TP203, TP31 to TP204, TP34 to TP205, TP37 to TP206, TP32 to TP207, TP35 to TP208, U20 to U201, U21 to U202, U22 to U203, U23 to U204, USB1 to USB201
Other:
- moved on the sheet: C201, C202, C203, C204, D201, J201, J202, R201, R202, R205, U203, U204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
