File: hardware/carrier-cm5/lte.kicad_sch (KiCad schematic)
At the start: 68 parts, among them J50 U.FL LTE, J51 U.FL GNSS, J52 SIM8060-6-0-14-00-A, J53 A7670E board, Q100 MMBT3904, Q101 MMBT3904, U50 A7670E-LASE, U51 TPS62933DRLR, U52 TXS0104EPW, U53 SP0504BAHT

Commit message: Updated schematic on CM5 carrier
Parts:
- D801: renamed from D101; value BLUE -> GREEN
- renumbered C100 to C801, C105 to C802, C111 to C803, C101 to C804, C112 to C805, C106 to C806, C107 to C807, C102 to C808, C108 to C809, C103 to C810, C109 to C811, C110 to C812, C104 to C813, C114 to C814, C118 to C815, C119 to C816, C115 to C817, C120 to C818, C121 to C819, C113 to C820, C122 to C821, C116 to C822, C117 to C823, D100 to D802, J53 to J801, J50 to J802, J52 to J803, J51 to J804, JP50 to JP801, JP51 to JP802, L100 to L801, Q101 to Q801, Q100 to Q802, R103 to R801, R104 to R802, R100 to R803, R107 to R804, R105 to R805, R101 to R806, R106 to R807, R102 to R808, R117 to R809, R118 to R810, R119 to R811, R120 to R812, R114 to R813, R112 to R814, R115 to R815, R116 to R816, R111 to R817, R110 to R818, R109 to R819, R108 to R820, R113 to R821, TP70 to TP801, TP71 to TP802, TP72 to TP803, TP73 to TP804, TP74 to TP805, TP75 to TP806, TP76 to TP807, TP77 to TP808, TP78 to TP809, U51 to U801, U52 to U802, U50 to U803, U53 to U804
Other:
- note added: "A7670E LTE"
- note removed: "A7670E"
- company: AAC -> (none)
- moved on the sheet: C803, C804, C805, C808, C810, C813, C814, C815, C816, C817, C818, C819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
