File: hardware/carrier-cm5/m2.kicad_sch (KiCad schematic)
At the start: 26 parts, among them J8 M.2 M-key, U24 ASEK-32.768KHZ-L-R-T, U8 AP3441SHE-7B

Commit message: Updated schematic on CM5 carrier
Parts:
- renumbered C4 to C401, C6 to C402, C10 to C403, C11 to C404, C14 to C405, C15 to C406, C16 to C407, C17 to C408, C60 to C409, C61 to C410, C62 to C411, C77 to C412, D7 to D401, H7 to H401, J8 to J401, L1 to L401, R14 to R401, R15 to R402, R16 to R403, R53 to R404, TP38 to TP401, TP39 to TP402, TP40 to TP403, TP41 to TP404, U8 to U401, U24 to U402
Other:
- moved on the sheet: U402
