File: hardware/carrier-cm5/periph.kicad_sch (KiCad schematic)
At the start: 27 parts, among them J60 J-CAN, J61 J-CAN, J62 J-NOSE, J63 J-SWDREC, U60 MCP251863T-E/SS, U61 LSM6DSV16X, Y60 40MHz ABM8

Commit message: Updated schematic on CM5 carrier
Parts:
- renumbered C132 to C901, C133 to C902, C134 to C903, C135 to C904, C130 to C905, C131 to C906, C136 to C907, C137 to C908, D60 to D901, J63 to J901, J60 to J902, J61 to J903, J62 to J904, R131 to R901, R130 to R902, R132 to R903, TP80 to TP901, TP82 to TP902, TP84 to TP903, TP86 to TP904, TP81 to TP905, TP83 to TP906, TP85 to TP907, TP87 to TP908, U60 to U901, U61 to U902, Y60 to Y901
Other:
- company: AAC -> (none)

Commit message: carrier: xh can and sysctl connectors, io mcu wiring tidy
Parts:
- J902, J903: footprint Connector_JST:JST_GH_SM04B-GHS-TB_1x04-1MP_P1.25mm_Horizontal -> Connector_JST:JST_XH_S4B-XH-A-1_1x04_P2.50mm_Horizontal
Changed lines of the file:
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@@
 			)
 		)
-		(property "Footprint" "Connector_JST:JST_GH_SM04B-GHS-TB_1x04-1MP_P1.25mm_Horizontal"
+		(property "Footprint" "Connector_JST:JST_XH_S4B-XH-A-1_1x04_P2.50mm_Horizontal"
 			(at 190.5 33.02 0)
 			(hide yes)
@@
 			)
 		)
-		(property "Footprint" "Connector_JST:JST_GH_SM04B-GHS-TB_1x04-1MP_P1.25mm_Horizontal"
+		(property "Footprint" "Connector_JST:JST_XH_S4B-XH-A-1_1x04_P2.50mm_Horizontal"
 			(at 190.5 58.42 0)
 			(hide yes)
