File: hardware/nose-board/nose-board.kicad_sch (KiCad schematic)
At the start: 0 parts

Commit message: nose board: tof, magnetometer, level shifting, test points
Parts:
- added C1, C3, C4: 1u, Capacitor_SMD:C_0603_1608Metric, symbol Device:C
- added C10, C6, C8: 100n, Capacitor_SMD:C_0603_1608Metric, symbol Device:C
- added C2: 10u, Capacitor_SMD:C_0805_2012Metric, symbol Device:C
- added C5, C7, C9: 4.7u, Capacitor_SMD:C_0805_2012Metric, symbol Device:C
- added D1: GREEN, LED_SMD:LED_0603_1608Metric, symbol Device:LED
- added H1, H2, H3, H4: M2, MountingHole:MountingHole_2.2mm_M2, symbol Mechanical:MountingHole
- added H5, H6, H7, H8: M3, MountingHole:MountingHole_3.2mm_M3_DIN965_Pad_TopBottom, symbol Mechanical:MountingHole
- added IC1: MMC5983MA, nose-board:MMC5983MA, symbol nose-board:MMC5983MA
- added J1: J-NOSE, Connector_JST:JST_GH_SM08B-GHS-TB_1x08-1MP_P1.25mm_Horizontal, symbol Connector_Generic:Conn_01x08
- added Q1, Q2: BSS138, Package_TO_SOT_SMD:SOT-23, symbol Transistor_FET:BSS138
- added R1, R2: 2.2k, Resistor_SMD:R_0603_1608Metric, symbol Device:R
- added R10, R11, R12, R13, R14: 47k, Resistor_SMD:R_0603_1608Metric, symbol Device:R
- added R3: 100k, Resistor_SMD:R_0603_1608Metric, symbol Device:R
- added R4: 1k, Resistor_SMD:R_0603_1608Metric, symbol Device:R
- added R5, R7: 4.7k, Resistor_SMD:R_0603_1608Metric, symbol Device:R
- added R6: 200k, Resistor_SMD:R_0603_1608Metric, symbol Device:R
- added R8, R9: 10k, Resistor_SMD:R_0603_1608Metric, symbol Device:R
- added TP1: 3V3, TestPoint:TestPoint_Pad_D2.0mm, symbol Connector:TestPoint
- added TP2: 1V8, TestPoint:TestPoint_Pad_D2.0mm, symbol Connector:TestPoint
- added TP3: GND, TestPoint:TestPoint_Pad_D2.0mm, symbol Connector:TestPoint
- added TP4: SDA_1V8, TestPoint:TestPoint_Pad_D2.0mm, symbol Connector:TestPoint
- added TP5: SCL_1V8, TestPoint:TestPoint_Pad_D2.0mm, symbol Connector:TestPoint
- added TP6: INT, TestPoint:TestPoint_Pad_D2.0mm, symbol Connector:TestPoint
- added U1: PCA9306DCUR, Package_SO:VSSOP-8_2.3x2mm_P0.5mm, symbol Interface:PCA9306
- added U2: TLV75518PDBVR, Package_TO_SOT_SMD:SOT-23-5, symbol Regulator_Linear:TLV75518PDBV
- added U3: VL53L8CXV0GC_1, nose-board:VL53L8CXV0GC1, symbol nose-board:VL53L8CXV0GC_1
Connections:
- new net: D1.2 (A), R4.2
- new net +1V8: C10.1, C4.1, C7.1, C8.1, C9.1, Q1.1 (G), Q2.1 (G), R1.1, R12.1, R13.1, R14.1, R2.1, TP2.1, U1.2 (VREF1), U2.5 (OUT), U3.A3 (IOVDD), U3.B7 (CORE_1V8)
- new net +3V3: C1.1, C3.1, C5.1, C6.1, IC1.13 (VDDIO), IC1.2 (VDD), IC1.4 (SPI_CS), J1.1 (Pin_1), R5.1, R6.1, R7.1, R8.1, R9.1, TP1.1, U2.1 (IN), U2.3 (EN), U3.C4 (AVDD)
- new net GND: C1.2, C10.2, C2.2, C3.2, C4.2, C5.2, C6.2, C7.2, C8.2, C9.2, D1.1 (K), IC1.11 (GND_2), IC1.9 (GND_1), J1.2 (Pin_2), R10.2, R11.2, R3.2, TP3.1, U1.1 (GND), U2.2 (GND), U3.A6 (RSVD1), U3.A7 (RSVD2), U3.B4 (GND_1), U3.C3 (GND_2), U3.C6 (RSVD3), U3.C7 (GND_3)
- new net I2C_SCL: IC1.1 (SCL/SPI_SCK), J1.4 (Pin_4), R7.2, U1.6 (SCL2)
- new net I2C_SDA: IC1.16 (SDA/SPI_SDI), J1.3 (Pin_3), R5.2, U1.5 (SDA2)
- new net LED: J1.8 (Pin_8), R4.1
- new net MAG_CAP: C2.1, IC1.10 (CAP)
- new net MAG_INT: IC1.15 (INT), J1.7 (Pin_7), R3.1
- new net PCA_EN: R6.2, U1.7 (VREF2), U1.8 (EN)
- new net TOF_INT: J1.6 (Pin_6), Q2.3 (D), R9.2
- new net TOF_INT_1V8: Q2.2 (S), R13.2, TP6.1, U3.1 (GPIO1_1), U3.A1 (GPIO1_2)
- new net TOF_LPN: J1.5 (Pin_5), Q1.3 (D), R8.2
- new net TOF_LPN_1V8: Q1.2 (S), R14.2, U3.A2 (LPN)
- new net TOF_NCS: R11.1, U3.C2 (NCS)
- new net TOF_SCL: R2.2, TP5.1, U1.3 (SCL1), U3.A5 (SCL/MCLK)
- new net TOF_SDA: R1.2, TP4.1, U1.4 (SDA1), U3.A4 (SDA/MOSI)
- new net TOF_SPI_I2C_N: R10.1, U3.C1 (SPI_I2C_N)
- new net TOF_SYNC: R12.2, U3.B1 (GPIO2)
- no-connect marks 0 -> 9
Other:
- note added: "1.8V LDO"
- note added: "Board Mounting Holes"
- note added: "Connector"
- note added: "Level Shifting"
- note added: "Magnetometer"
- note added: "Raspberry Pi Camera Mount"
- note added: "Test Points"
- note added: "ToF Sensor"

Commit message: Full placement of nose board PCB
Parts:
- removed H7, H8: M3, MountingHole:MountingHole_3.2mm_M3_DIN965_Pad_TopBottom, symbol Mechanical:MountingHole
- added J2: J-NOSE, Connector_JST:JST_GH_SM08B-GHS-TB_1x08-1MP_P1.25mm_Horizontal, symbol Connector_Generic:Conn_01x08
- H5, H6: value M3 -> M2; footprint MountingHole:MountingHole_3.2mm_M3_DIN965_Pad_TopBottom -> MountingHole:MountingHole_2.2mm_M2_Pad_TopBottom
Connections:
- net +3V3: now also J1.8 (Pin_8), J2.1 (Pin_1); no longer J1.1 (Pin_1)
- net GND: now also J1.7 (Pin_7), J2.2 (Pin_2); no longer J1.2 (Pin_2)
- net I2C_SCL: now also J1.5 (Pin_5), J2.4 (Pin_4); no longer J1.4 (Pin_4)
- net I2C_SDA: now also J1.6 (Pin_6), J2.3 (Pin_3); no longer J1.3 (Pin_3)
- net LED: now also J1.1 (Pin_1), J2.8 (Pin_8); no longer J1.8 (Pin_8)
- net MAG_INT: now also J1.2 (Pin_2), J2.7 (Pin_7); no longer J1.7 (Pin_7)
- net TOF_INT: now also J1.3 (Pin_3), J2.6 (Pin_6); no longer J1.6 (Pin_6)
- net TOF_LPN: now also J1.4 (Pin_4), J2.5 (Pin_5); no longer J1.5 (Pin_5)
Other:
- note removed: "Test Points"
- moved on the sheet: C1, C10, C2, C3, C4, C5, C6, C7, C8, C9, D1, H1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
