File: hardware/power-board/charger.kicad_sch (KiCad schematic)
At the start: 0 parts

Commit message: Added more ICs for power board
Parts:
- added D1: SMBJ20A, power-board:DIOM5436X244N, symbol power-board:SMBJ20A
- added IC3: CYPD3177-24LQXQ, power-board:QFN50P400X400X60-25N-D, symbol power-board:CYPD3177-24LQXQ
- added IC4: BQ25798RQMR, power-board:BQ25798RQMR, symbol power-board:BQ25798RQMR
- added P1: USB_C_Plug_USB2.0, symbol Connector:USB_C_Plug_USB2.0
- added Q1: BSS138-7-F, power-board:SOT96P240X115-3N, symbol power-board:BSS138-7-F
Connections:
- new net: P1.A1 (GND), P1.A12 (GND), P1.B1 (GND), P1.B12 (GND)
- new net: P1.A4 (VBUS), P1.A9 (VBUS), P1.B4 (VBUS), P1.B9 (VBUS)

Commit message: draw power board bms, charger and mcu circuits
Parts:
- removed P1: USB_C_Plug_USB2.0, symbol Connector:USB_C_Plug_USB2.0
- added C401, C402, C412, C413, C414, C416, C417, C418, C419, C420, C421, C422: 10u 25V, Capacitor_SMD:C_0805_2012Metric, symbol Device:C
- added C403, C406: 1u, Capacitor_SMD:C_0805_2012Metric, symbol Device:C
- added C404, C405: 100n, Capacitor_SMD:C_0805_2012Metric, symbol Device:C
- added C407: 4.7u 10V, Capacitor_SMD:C_0805_2012Metric, symbol Device:C
- added C408, C409: 47n, Capacitor_SMD:C_0805_2012Metric, symbol Device:C
- added C410: 1n 50V, Capacitor_SMD:C_0805_2012Metric, symbol Device:C
- added C411, C415: 100n 50V, Capacitor_SMD:C_0805_2012Metric, symbol Device:C
- added D401: CHG, LED_SMD:LED_0603_1608Metric, symbol Device:LED
- added J401: USB4125-GF-A, Connector_USB:USB_C_Receptacle_GCT_USB4125-xx-x_6P_TopMnt_Horizontal, symbol Connector:USB_C_Receptacle_PowerOnly_6P
- added L401: 1u, Inductor_SMD:L_Coilcraft_XAL5030-XXX, symbol Device:L
- added R401, R402: 100k, Resistor_SMD:R_0603_1608Metric, symbol Device:R
- added R403, R405, R406, R408: 5.1k, Resistor_SMD:R_0603_1608Metric, symbol Device:R
- added R404: 1k, Resistor_SMD:R_0603_1608Metric, symbol Device:R
- added R407: 10k, Resistor_SMD:R_0603_1608Metric, symbol Device:R
- added R409: 7.5k, Resistor_SMD:R_0603_1608Metric, symbol Device:R
- added R410: 2.2k, Resistor_SMD:R_0603_1608Metric, symbol Device:R
- added R411: 17.4k, Resistor_SMD:R_0603_1608Metric, symbol Device:R
- added R412: 100, Resistor_SMD:R_0603_1608Metric, symbol Device:R
Connections:
- net BCR_VMIN: now reaches IC3.1 (VBUS_MIN)
- net BCR_VMIN: now also R403.2, R404.1
- net VBUS: now reaches IC3.11 (VDC_OUT)
- net VBUS: now also D1.1 (K), IC3.18 (VBUS_IN), IC4.2 (VBUS_1), IC4.3 (VBUS_2), IC4.31 (VAC1_2), IC4.8 (VAC2), IC4.9 (VAC1_1), C401.1, C402.1, J401.A9 (VBUS), J401.B9 (VBUS), R401.1
- net CC2: now reaches IC3.14 (CC2)
- net CC2: now also J401.B5 (CC2)
- net CC1: now reaches IC3.15 (CC1)
- net CC1: now also J401.A5 (CC1)
- net GND: now reaches IC3.19 (GND_1)
- net GND: now also D1.2 (A), IC3.22 (GND_2), IC3.25 (GND_3), IC3.6 (ISNK_FINE), IC4.10 (ACDRV2), IC4.11 (ACDRV1), IC4.27 (GND), Q1.2 (S), C401.2, C402.2, C403.2, C404.2, C405.2, C406.2, C407.2, C410.2, C411.2, C412.2, C413.2, C414.2, C415.2, C416.2, C417.2, C418.2, C419.2, C420.2, C421.2, C422.2, J401.A12 (GND), J401.B12 (GND), J401.SH (SHIELD), R402.2, R404.2, R406.2, R407.2, R409.2, R411.2
- net VDDD: now reaches IC3.2 (VBUS_MAX)
- net VDDD: now also IC3.23 (VDDD), C403.1, C404.1, C405.1, R403.1, R405.1
- net VCCD: now reaches IC3.24 (VCCD)
- net VCCD: now also C406.1
- net BCR_ISNK: now reaches IC3.5 (ISNK_COARSE)
- net BCR_ISNK: now also R405.2, R406.1
- net WAKE_G: now reaches Q1.1 (G)
- net WAKE_G: now also R401.2, R402.1
- net TS2_WAKE: now reaches Q1.3 (D)
- net CHG_STAT: now reaches IC4.1 (STAT_1)
- net CHG_STAT: now also IC4.30 (STAT_2), D401.1 (K)
- net CHG_CE: now reaches IC4.13 (~{CE})
- net CHG_CE: now also R407.1
- net I2C_SCL: now reaches IC4.14 (SCL)
- net I2C_SDA: now reaches IC4.15 (SDA)
- net CHG_TS: now reaches IC4.16 (TS_1)
- net CHG_TS: now also IC4.32 (TS_2), R408.2, R409.1
- net REGN: now reaches IC4.17 (ILIM_HIZ)
- net REGN: now also IC4.5 (REGN), C407.1, R408.1, R410.1
- net CHG_BATP: now reaches IC4.18 (BATP)
- net CHG_BATP: now also R412.1
- net CHG_BTST2: now reaches IC4.19 (BTST2)
- net CHG_BTST2: now also C409.1
- net CHG_PROG: now reaches IC4.20 (PROG)
- net CHG_PROG: now also R411.1
- net CHG_INT: now reaches IC4.21 (~{INT})
- net PACK+: now reaches IC4.22 (BAT_1)
- net PACK+: now also IC4.23 (BAT_2), C421.1, C422.1, R412.2
- net CHG_SDRV: now reaches IC4.24 (SDRV_1)
- net CHG_SDRV: now also IC4.33 (SDRV_2), C410.1
- net CHG_SYS: now reaches IC4.25 (SYS)
- net CHG_SYS: now also C415.1, C416.1, C417.1, C418.1, C419.1, C420.1
- net CHG_SW2: now reaches IC4.26 (SW2)
- net CHG_SW2: now also C409.2, L401.2
- net CHG_SW1: now reaches IC4.28 (SW1)
- net CHG_SW1: now also C408.2, L401.1
- net CHG_PMID: now reaches IC4.29 (PMID)
- net CHG_PMID: now also C411.1, C412.1, C413.1, C414.1
- net CHG_BTST1: now reaches IC4.4 (BTST1)
- net CHG_BTST1: now also C408.1
- new net CHG_LED: D401.2 (A), R410.2
- no-connect marks 0 -> 15
Other:
- note added: "Charger"
- note added: "PD Controller"
- note added: "USB-C Input"
- note added: "Wake"
- moved on the sheet: D1, IC3, IC4, Q1

Commit message: Reset annotations for power board
Parts:
- D302: renamed from D401; value CHG -> GREEN
- renumbered C401 to C301, C402 to C302, C407 to C303, C408 to C304, C415 to C305, C416 to C306, C409 to C307, C417 to C308, C418 to C309, C410 to C310, C419 to C311, C420 to C312, C411 to C313, C412 to C314, C421 to C315, C403 to C316, C413 to C317, C422 to C318, C404 to C319, C414 to C320, C405 to C321, C406 to C322, D1 to D301, IC4 to IC301, IC3 to IC302, J401 to J301, L401 to L301, Q1 to Q301, R407 to R301, R410 to R302, R401 to R303, R408 to R304, R402 to R305, R409 to R306, R403 to R307, R404 to R308, R405 to R309, R406 to R310, R411 to R311, R412 to R312
Other:
- moved on the sheet: C316, C319, C321, C322, IC302, Q301, R303, R305, R307, R308, R309, R310

Commit message: power board: test points
Parts:
- added TP401: VBUS, TestPoint:TestPoint_Pad_D2.0mm, symbol Connector:TestPoint
- added TP402: REGN, TestPoint:TestPoint_Pad_D2.0mm, symbol Connector:TestPoint
- added TP403: SYS, TestPoint:TestPoint_Pad_D2.0mm, symbol Connector:TestPoint
- added TP404: VDDD, TestPoint:TestPoint_Pad_D2.0mm, symbol Connector:TestPoint
- added TP405: STAT, TestPoint:TestPoint_Pad_D2.0mm, symbol Connector:TestPoint
- added TP406: INT, TestPoint:TestPoint_Pad_D2.0mm, symbol Connector:TestPoint
Connections:
- net CHG_INT: now also TP406.1
- net CHG_STAT: now also TP405.1
- net CHG_SYS: now also TP403.1
- net REGN: now also TP402.1
- net VBUS: now also TP401.1
- net VDDD: now also TP404.1
Other:
- note added: "Test Points"

Commit message: power board: amrm inductor, sot-223 for q204, 2.2k i2c pull-ups, 50 v charger caps, xh connectors
Parts:
- C301, C302, C314: value 10u 25V -> 10u 50V; footprint Capacitor_SMD:C_0805_2012Metric -> Capacitor_SMD:C_1206_3216Metric
