Commit message: Added fix to URDF

File: software/ros2_ws/src/vector_description/urdf/vector_cad_raw.urdf.xacro (robot description, xacro)
@@ -1,10 +1,8 @@
 <?xml version='1.0' encoding='utf-8'?>
-<!-- Generated by software/tools/cad_urdf.py from vector_cad_raw.urdf.xacro. Do not edit. -->
 <robot xmlns:xacro="http://www.ros.org/wiki/xacro" name="V.E.C.T.O.R.">
    <xacro:include filename="$(find vector_description)/urdf/vector_cad_materials.xacro" />
-   <link name="base_link" />
-   <joint name="base_link_cad_joint" type="fixed">
-      <origin xyz="1.57833862e-11 1.97295883e-14 -0.00929105671" rpy="0 -0 0" />
-      <parent link="base_link" />
+   <link name="dummy_link" />
+   <joint name="dummy_link_joint" type="fixed">
+      <parent link="dummy_link" />
       <child link="base_linkv8_1" />
    </joint>
@@ -12,6 +10,6 @@
       <inertial>
          <origin xyz="-0.0018772313854202062 -6.831789961107053e-06 0.0014778649263716926" rpy="0.0 0.0 3.141592653589793" />
-         <mass value="0.255341973" />
-         <inertia ixx="0.000388154123" iyy="0.000988083423" izz="0.00124816676" ixy="-8.90616742e-08" iyz="1.10355968e-07" ixz="3.85873541e-07" />
+         <mass value="1.2686581992949608" />
+         <inertia ixx="0.001928531" iyy="0.0049092599999999995" izz="0.0062014755" ixy="-4.4250000000000005e-07" iyz="5.483e-07" ixz="1.9172e-06" />
       </inertial>
       <visual>
@@ -95,6 +93,6 @@
       <inertial>
          <origin xyz="-0.00010921397547406064 1.1301399740667222e-05 0.021399999443451643" rpy="0.0 0.0 3.141592653589793" />
-         <mass value="0.0505988624" />
-         <inertia ixx="4.464705e-05" iyy="0.000154271364" izz="0.000198842515" ixy="1.72890346e-08" iyz="-0" ixz="0" />
+         <mass value="0.2513987840352954" />
+         <inertia ixx="0.00022182740000000004" iyy="0.0007664922000000001" izz="0.0009879425" ixy="8.59e-08" iyz="-0.0" ixz="0.0" />
       </inertial>
       <visual>
@@ -115,6 +113,6 @@
       <inertial>
          <origin xyz="-0.00020660958419582487 0.0006267751670009789 0.022000000000000002" rpy="0.0 0.0 3.141592653589793" />
-         <mass value="0.0172035601" />
-         <inertia ixx="2.34144852e-05" iyy="6.64560098e-05" izz="8.98539709e-05" ixy="-8.77534236e-09" iyz="0" ixz="-0" />
+         <mass value="0.08547532263943959" />
+         <inertia ixx="0.00011633410000000001" iyy="0.00033018450000000003" izz="0.0004464365" ixy="-4.3600000000000007e-08" iyz="0.0" ixz="-0.0" />
       </inertial>
       <visual>
@@ -135,6 +133,6 @@
       <inertial>
          <origin xyz="0.0893150541355548 -0.03263535407427847 -0.004978940218193806" rpy="-1.5707963267948966 0.7853981633974585 -1.5707963267948966" />
-         <mass value="0.0484640241" />
-         <inertia ixx="1.06611554e-05" iyy="1.06608937e-05" izz="9.14877746e-06" ixy="-2.9942233e-06" iyz="2.23127168e-07" ixz="2.22744757e-07" />
+         <mass value="0.2407919102798682" />
+         <inertia ixx="5.29696e-05" iyy="5.2968300000000006e-05" izz="4.54554e-05" ixy="-1.4876700000000003e-05" iyz="1.1086e-06" ixz="1.1067000000000001e-06" />
       </inertial>
    </link>
@@ -142,6 +140,6 @@
       <inertial>
          <origin xyz="0.08931505413555481 -0.03263535407427847 -0.004978940218193913" rpy="-1.5707963267948966 0.0 -1.5707963267948966" />
-         <mass value="0.0484640241" />
-         <inertia ixx="1.36552378e-05" iyy="7.66681132e-06" izz="9.14877746e-06" ixy="1.40888524e-10" iyz="3.1528839e-07" ixz="-2.61650116e-10" />
+         <mass value="0.2407919102798682" />
+         <inertia ixx="6.78456e-05" iyy="3.80923e-05" izz="4.54554e-05" ixy="7.000000000000001e-10" iyz="1.5665e-06" ixz="-1.3e-09" />
       </inertial>
    </link>
@@ -149,6 +147,6 @@
       <inertial>
          <origin xyz="0.08931505413555481 -0.03263535407427835 -0.004978940218193806" rpy="1.5707963267948966 -0.7853981633974496 1.5707963267948966" />
-         <mass value="0.0484640241" />
-         <inertia ixx="1.06611554e-05" iyy="1.06608937e-05" izz="9.14877746e-06" ixy="-2.9942233e-06" iyz="-2.23127168e-07" ixz="-2.22744757e-07" />
+         <mass value="0.2407919102798682" />
+         <inertia ixx="5.29696e-05" iyy="5.2968300000000006e-05" izz="4.54554e-05" ixy="-1.4876700000000003e-05" iyz="-1.1086e-06" ixz="-1.1067000000000001e-06" />
       </inertial>
    </link>
@@ -156,6 +154,6 @@
       <inertial>
          <origin xyz="0.08931505413555481 -0.03263535407427841 -0.004978940218193948" rpy="1.5707963267948966 0.0 1.5707963267948966" />
-         <mass value="0.0484640241" />
-         <inertia ixx="1.36552378e-05" iyy="7.66681132e-06" izz="9.14877746e-06" ixy="1.40888524e-10" iyz="-3.1528839e-07" ixz="2.61650116e-10" />
+         <mass value="0.2407919102798682" />
+         <inertia ixx="6.78456e-05" iyy="3.80923e-05" izz="4.54554e-05" ixy="7.000000000000001e-10" iyz="-1.5665e-06" ixz="1.3e-09" />
       </inertial>
    </link>
@@ -163,6 +161,6 @@
       <inertial>
          <origin xyz="0.08931505413555484 -0.032635354074278436 -0.0049789402181938235" rpy="1.5707963267948966 0.7853981633974532 1.5707963267948966" />
-         <mass value="0.0484640241" />
-         <inertia ixx="1.06608937e-05" iyy="1.06611554e-05" izz="9.14877746e-06" ixy="2.9942233e-06" iyz="-2.22744757e-07" ixz="2.23127168e-07" />
+         <mass value="0.2407919102798682" />
+         <inertia ixx="5.2968300000000006e-05" iyy="5.29696e-05" izz="4.54554e-05" ixy="1.4876700000000003e-05" iyz="-1.1067000000000001e-06" ixz="1.1086e-06" />
       </inertial>
    </link>
@@ -170,6 +168,6 @@
       <inertial>
          <origin xyz="0.009496810901016462 0.008593417004839416 -0.007069952519590395" rpy="-1.5707963267948966 0.7853981633974318 0.0" />
-         <mass value="0.00327439061" />
-         <inertia ixx="1.23452563e-06" iyy="1.23440487e-06" izz="1.47377447e-06" ixy="-4.79906567e-07" iyz="2.06703592e-08" ixz="2.04489629e-08" />
+         <mass value="0.016268702078190932" />
+         <inertia ixx="6.1337e-06" iyy="6.1331e-06" izz="7.3224e-06" ixy="-2.3844e-06" iyz="1.027e-07" ixz="1.016e-07" />
       </inertial>
       <visual>
@@ -190,6 +188,6 @@
       <inertial>
          <origin xyz="7.847128724591812e-10 0.018862565434485133 0.00019573987745458155" rpy="-1.5707963267948966 0.7853981633974323 0.0" />
-         <mass value="0.0451896335" />
-         <inertia ixx="8.98764124e-06" iyy="8.98764124e-06" izz="7.5342151e-06" ixy="-2.44391272e-06" iyz="4.13205914e-08" ixz="4.13205914e-08" />
+         <mass value="0.2245232082016773" />
+         <inertia ixx="4.46548e-05" iyy="4.46548e-05" izz="3.74335e-05" ixy="-1.2142500000000001e-05" iyz="2.0530000000000002e-07" ixz="2.0530000000000002e-07" />
       </inertial>
       <visual>
@@ -252,6 +250,6 @@
       <inertial>
          <origin xyz="0.009496810901016452 0.008593417004839416 -0.0070699525195903855" rpy="-1.5707963267948966 0.0 0.0" />
-         <mass value="0.00327439061" />
-         <inertia ixx="1.71437182e-06" iyy="7.54558681e-07" izz="1.47377447e-06" ixy="6.0380796e-11" iyz="2.90632898e-08" ixz="-1.61015456e-10" />
+         <mass value="0.016268702078190932" />
+         <inertia ixx="8.5178e-06" iyy="3.749000000000001e-06" izz="7.3224e-06" ixy="3.0000000000000005e-10" iyz="1.4440000000000002e-07" ixz="-8e-10" />
       </inertial>
       <visual>
@@ -272,6 +270,6 @@
       <inertial>
          <origin xyz="7.847128391524905e-10 0.018862565434485133 0.00019573987745458155" rpy="-1.5707963267948966 0.0 0.0" />
-         <mass value="0.0451896335" />
-         <inertia ixx="1.1431554e-05" iyy="6.54372852e-06" izz="7.5342151e-06" ixy="0" iyz="5.84284836e-08" ixz="-0" />
+         <mass value="0.2245232082016773" />
+         <inertia ixx="5.67973e-05" iyy="3.25123e-05" izz="3.74335e-05" ixy="0.0" iyz="2.903e-07" ixz="-0.0" />
       </inertial>
       <visual>
@@ -334,6 +332,6 @@
       <inertial>
          <origin xyz="0.009496810901016466 0.008593417004839416 -0.0070699525195903595" rpy="1.5707963267948966 -0.7853981633974217 3.141592653589793" />
-         <mass value="0.00327439061" />
-         <inertia ixx="1.23452563e-06" iyy="1.23440487e-06" izz="1.47377447e-06" ixy="-4.79906567e-07" iyz="-2.06703592e-08" ixz="-2.04489629e-08" />
+         <mass value="0.016268702078190932" />
+         <inertia ixx="6.1337e-06" iyy="6.1331e-06" izz="7.3224e-06" ixy="-2.3844e-06" iyz="-1.027e-07" ixz="-1.016e-07" />
       </inertial>
       <visual>
@@ -354,6 +352,6 @@
       <inertial>
          <origin xyz="7.847128458138286e-10 0.01886256543448514 0.00019573987745458155" rpy="1.5707963267948966 -0.7853981633974225 -3.141592653589793" />
-         <mass value="0.0451896335" />
-         <inertia ixx="8.98764124e-06" iyy="8.98764124e-06" izz="7.5342151e-06" ixy="-2.44391272e-06" iyz="-4.13205914e-08" ixz="-4.13205914e-08" />
+         <mass value="0.2245232082016773" />
+         <inertia ixx="4.46548e-05" iyy="4.46548e-05" izz="3.74335e-05" ixy="-1.2142500000000001e-05" iyz="-2.0530000000000002e-07" ixz="-2.0530000000000002e-07" />
       </inertial>
       <visual>
@@ -416,6 +414,6 @@
       <inertial>
          <origin xyz="0.009496810901016452 0.008593417004839416 -0.0070699525195903595" rpy="1.5707963267948966 0.0 3.141592653589793" />
-         <mass value="0.00327439061" />
-         <inertia ixx="1.71437182e-06" iyy="7.54558681e-07" izz="1.47377447e-06" ixy="6.0380796e-11" iyz="-2.90632898e-08" ixz="1.61015456e-10" />
+         <mass value="0.016268702078190932" />
+         <inertia ixx="8.5178e-06" iyy="3.749000000000001e-06" izz="7.3224e-06" ixy="3.0000000000000005e-10" iyz="-1.4440000000000002e-07" ixz="8e-10" />
       </inertial>
       <visual>
@@ -436,6 +434,6 @@
       <inertial>
          <origin xyz="7.847128347115984e-10 0.01886256543448514 0.000195739877454546" rpy="1.5707963267948966 0.0 3.141592653589793" />
-         <mass value="0.0451896335" />
-         <inertia ixx="1.1431554e-05" iyy="6.54372852e-06" izz="7.5342151e-06" ixy="0" iyz="-5.84284836e-08" ixz="0" />
+         <mass value="0.2245232082016773" />
+         <inertia ixx="5.67973e-05" iyy="3.25123e-05" izz="3.74335e-05" ixy="0.0" iyz="-2.903e-07" ixz="0.0" />
       </inertial>
       <visual>
@@ -498,6 +496,6 @@
       <inertial>
          <origin xyz="0.009496810901016471 0.008593417004839425 -0.007069952519590377" rpy="1.5707963267948966 0.7853981633974825 3.141592653589793" />
-         <mass value="0.00327439061" />
-         <inertia ixx="1.23440487e-06" iyy="1.23452563e-06" izz="1.47377447e-06" ixy="4.79906567e-07" iyz="-2.04489629e-08" ixz="2.06703592e-08" />
+         <mass value="0.016268702078190932" />
+         <inertia ixx="6.1331e-06" iyy="6.1337e-06" izz="7.3224e-06" ixy="2.3844e-06" iyz="-1.016e-07" ixz="1.027e-07" />
       </inertial>
       <visual>
@@ -518,6 +516,6 @@
       <inertial>
          <origin xyz="7.847128280502602e-10 0.018862565434485168 0.0001957398774545638" rpy="1.5707963267948966 0.7853981633974829 3.141592653589793" />
-         <mass value="0.0451896335" />
-         <inertia ixx="8.98764124e-06" iyy="8.98764124e-06" izz="7.5342151e-06" ixy="2.44391272e-06" iyz="-4.13205914e-08" ixz="4.13205914e-08" />
+         <mass value="0.2245232082016773" />
+         <inertia ixx="4.46548e-05" iyy="4.46548e-05" izz="3.74335e-05" ixy="1.2142500000000001e-05" iyz="-2.0530000000000002e-07" ixz="2.0530000000000002e-07" />
       </inertial>
       <visual>
@@ -580,6 +578,6 @@
       <inertial>
          <origin xyz="0.009496810901016452 0.008593417004839399 -0.007069952519590377" rpy="-1.5707963267948966 -0.7853981633974779 0.0" />
-         <mass value="0.00327439061" />
-         <inertia ixx="1.23440487e-06" iyy="1.23452563e-06" izz="1.47377447e-06" ixy="4.79906567e-07" iyz="2.04489629e-08" ixz="-2.06703592e-08" />
+         <mass value="0.016268702078190932" />
+         <inertia ixx="6.1331e-06" iyy="6.1337e-06" izz="7.3224e-06" ixy="2.3844e-06" iyz="1.016e-07" ixz="-1.027e-07" />
       </inertial>
       <visual>
@@ -599,10 +597,10 @@
    <link name="FemurBracketv3_1">
       <inertial>
-         <origin xyz="-1.6862425e-05 -0.0139524957 0.0339670466" rpy="-3.14159265 -6.65280469e-33 2.37014352" />
-         <mass value="0.016897885" />
-         <inertia ixx="1.36308641e-05" iyy="1.36002913e-05" izz="3.26929808e-06" ixy="-5.78649295e-07" iyz="1.30301758e-07" ixz="1.26598402e-07" />
-      </inertial>
-      <visual>
-         <origin xyz="-0.0502774784 0.139072481 0.12131116" rpy="-3.14159265 -6.65280469e-33 2.37014352" />
+         <origin xyz="0.00015061611064049352 -0.025951347267356317 0.03396704662982687" rpy="-3.141592653589793 0.0 2.3701435180688293" />
+         <mass value="0.08395658588476052" />
+         <inertia ixx="6.77245e-05" iyy="6.757260000000001e-05" izz="1.62434e-05" ixy="-2.875e-06" iyz="6.473999999999999e-07" ixz="6.29e-07" />
+      </inertial>
+      <visual>
+         <origin xyz="-0.05010999991300913 0.12707362990603613 0.12131116015941817" rpy="-3.141592653589793 0.0 2.3701435180688293" />
          <geometry>
             <mesh filename="package://vector_description/meshes/FemurBracketv3_1__FemurBracketEndCap.stl" scale="0.001 0.001 0.001" />
@@ -611,5 +609,5 @@
       </visual>
       <visual>
-         <origin xyz="-0.0502774784 0.139072481 0.12131116" rpy="-3.14159265 -6.65280469e-33 2.37014352" />
+         <origin xyz="-0.05010999991300913 0.12707362990603613 0.12131116015941817" rpy="-3.141592653589793 0.0 2.3701435180688293" />
          <geometry>
             <mesh filename="package://vector_description/meshes/FemurBracketv3_1__FemurBracket.stl" scale="0.001 0.001 0.001" />
@@ -618,5 +616,5 @@
       </visual>
       <collision>
-         <origin xyz="-0.0502774784 0.139072481 0.12131116" rpy="-3.14159265 -6.65280469e-33 2.37014352" />
+         <origin xyz="-0.05010999991300913 0.12707362990603613 0.12131116015941817" rpy="-3.141592653589793 0.0 2.3701435180688293" />
          <geometry>
             <mesh filename="package://vector_description/meshes/FemurBracketv3_1.stl" scale="0.001 0.001 0.001" />
@@ -627,6 +625,6 @@
       <inertial>
          <origin xyz="-1.6766795655542843e-05 -0.013952514700698871 0.03396704662982684" rpy="3.141592653589793 0.0 0.013949027876495323" />
-         <mass value="0.016897885" />
-         <inertia ixx="1.4194237e-05" iyy="1.30369183e-05" izz="3.26929808e-06" ixy="1.52964683e-08" iyz="-1.81665688e-07" ixz="2.61650116e-09" />
+         <mass value="0.08395658588476052" />
+         <inertia ixx="7.05236e-05" iyy="6.477349999999999e-05" izz="1.62434e-05" ixy="7.6e-08" iyz="-9.025999999999999e-07" ixz="1.2999999999999999e-08" />
       </inertial>
       <visual>
@@ -653,10 +651,10 @@
    <link name="FemurBracketv3_1_0">
       <inertial>
-         <origin xyz="-1.6862456e-05 -0.0139524957 0.0339670466" rpy="-3.14159265 2.04338263e-33 -3.12764363" />
-         <mass value="0.016897885" />
-         <inertia ixx="1.4194237e-05" iyy="1.30369183e-05" izz="3.26929808e-06" ixy="1.52964683e-08" iyz="1.81665688e-07" ixz="-2.61650116e-09" />
-      </inertial>
-      <visual>
-         <origin xyz="-0.0213469772 0.0964116399 0.12131116" rpy="-3.14159265 2.04338263e-33 -3.12764363" />
+         <origin xyz="0.0001506161106404269 -0.025951347267356404 0.03396704662982693" rpy="-3.141592653589793 0.0 -3.1276436257132776" />
+         <mass value="0.08395658588476052" />
+         <inertia ixx="7.05236e-05" iyy="6.477349999999999e-05" izz="1.62434e-05" ixy="7.6e-08" iyz="9.025999999999999e-07" ixz="-1.2999999999999999e-08" />
+      </inertial>
+      <visual>
+         <origin xyz="-0.021179498624701143 0.08441278835583071 0.12131116015941867" rpy="-3.141592653589793 0.0 -3.1276436257132776" />
          <geometry>
             <mesh filename="package://vector_description/meshes/FemurBracketv3_1_0__FemurBracketEndCap.stl" scale="0.001 0.001 0.001" />
@@ -665,5 +663,5 @@
       </visual>
       <visual>
-         <origin xyz="-0.0213469772 0.0964116399 0.12131116" rpy="-3.14159265 2.04338263e-33 -3.12764363" />
+         <origin xyz="-0.021179498624701143 0.08441278835583071 0.12131116015941867" rpy="-3.141592653589793 0.0 -3.1276436257132776" />
          <geometry>
             <mesh filename="package://vector_description/meshes/FemurBracketv3_1_0__FemurBracket.stl" scale="0.001 0.001 0.001" />
@@ -672,5 +670,5 @@
       </visual>
       <collision>
-         <origin xyz="-0.0213469772 0.0964116399 0.12131116" rpy="-3.14159265 2.04338263e-33 -3.12764363" />
+         <origin xyz="-0.021179498624701143 0.08441278835583071 0.12131116015941867" rpy="-3.141592653589793 0.0 -3.1276436257132776" />
          <geometry>
             <mesh filename="package://vector_description/meshes/FemurBracketv3_1_0.stl" scale="0.001 0.001 0.001" />
@@ -680,10 +678,10 @@
    <link name="FemurBracketv3_1_1">
       <inertial>
-         <origin xyz="-1.68624752e-05 -0.0139524957 0.0339670466" rpy="3.14159265 -4.61263969e-32 -0.771449136" />
-         <mass value="0.016897885" />
-         <inertia ixx="1.36308641e-05" iyy="1.36002913e-05" izz="3.26929808e-06" ixy="-5.78649295e-07" iyz="-1.30301758e-07" ixz="-1.26598402e-07" />
-      </inertial>
-      <visual>
-         <origin xyz="-0.0241759471 0.110841621 0.12131116" rpy="3.14159265 -4.61263969e-32 -0.771449136" />
+         <origin xyz="0.00015061611064040914 -0.02595134726735642 0.03396704662982687" rpy="3.141592653589793 0.0 -0.7714491355209543" />
+         <mass value="0.08395658588476052" />
+         <inertia ixx="6.77245e-05" iyy="6.757260000000001e-05" izz="1.62434e-05" ixy="-2.875e-06" iyz="-6.473999999999999e-07" ixz="-6.29e-07" />
+      </inertial>
+      <visual>
+         <origin xyz="-0.02400846852429194 0.09884276952382713 0.12131116015941885" rpy="3.141592653589793 0.0 -0.7714491355209543" />
          <geometry>
             <mesh filename="package://vector_description/meshes/FemurBracketv3_1_1__FemurBracketEndCap.stl" scale="0.001 0.001 0.001" />
@@ -692,5 +690,5 @@
       </visual>
       <visual>
-         <origin xyz="-0.0241759471 0.110841621 0.12131116" rpy="3.14159265 -4.61263969e-32 -0.771449136" />
+         <origin xyz="-0.02400846852429194 0.09884276952382713 0.12131116015941885" rpy="3.141592653589793 0.0 -0.7714491355209543" />
          <geometry>
             <mesh filename="package://vector_description/meshes/FemurBracketv3_1_1__FemurBracket.stl" scale="0.001 0.001 0.001" />
@@ -699,5 +697,5 @@
       </visual>
       <collision>
-         <origin xyz="-0.0241759471 0.110841621 0.12131116" rpy="3.14159265 -4.61263969e-32 -0.771449136" />
+         <origin xyz="-0.02400846852429194 0.09884276952382713 0.12131116015941885" rpy="3.141592653589793 0.0 -0.7714491355209543" />
          <geometry>
             <mesh filename="package://vector_description/meshes/FemurBracketv3_1_1.stl" scale="0.001 0.001 0.001" />
@@ -708,6 +706,6 @@
       <inertial>
          <origin xyz="-1.676679565556505e-05 -0.013952514700698943 0.03396704662982689" rpy="-3.141592653589793 0.0 0.7993471912739496" />
-         <mass value="0.016897885" />
-         <inertia ixx="1.36002913e-05" iyy="1.36308641e-05" izz="3.26929808e-06" ixy="5.78649295e-07" iyz="-1.26598402e-07" ixz="1.30301758e-07" />
+         <mass value="0.08395658588476052" />
+         <inertia ixx="6.757260000000001e-05" iyy="6.77245e-05" izz="1.62434e-05" ixy="2.875e-06" iyz="-6.29e-07" ixz="6.473999999999999e-07" />
       </inertial>
       <visual>
@@ -735,6 +733,6 @@
       <inertial>
          <origin xyz="0.08931505413555484 -0.03263535407427843 -0.004978940218193806" rpy="-1.5707963267948966 -0.7853981633974498 -1.5707963267948966" />
-         <mass value="0.0484640241" />
-         <inertia ixx="1.06608937e-05" iyy="1.06611554e-05" izz="9.14877746e-06" ixy="2.9942233e-06" iyz="2.22744757e-07" ixz="-2.23127168e-07" />
+         <mass value="0.2407919102798682" />
+         <inertia ixx="5.2968300000000006e-05" iyy="5.29696e-05" izz="4.54554e-05" ixy="1.4876700000000003e-05" iyz="1.1067000000000001e-06" ixz="-1.1086e-06" />
       </inertial>
    </link>
@@ -742,6 +740,6 @@
       <inertial>
          <origin xyz="0.0887805528859608 -0.031884925293127045 0.03099564848668308" rpy="1.5707963267948966 -0.7853981633974496 1.5707963267948966" />
-         <mass value="0.0398443972" />
-         <inertia ixx="2.83815705e-05" iyy="2.99657412e-05" izz="2.81289574e-05" ixy="1.06831742e-06" iyz="-5.2744638e-07" ixz="-5.8760578e-07" />
+         <mass value="0.19796557769577772" />
+         <inertia ixx="0.00014101290000000002" iyy="0.00014888380000000002" izz="0.0001397578" ixy="5.3079000000000005e-06" iyz="-2.6206e-06" ixz="-2.9194999999999997e-06" />
       </inertial>
    </link>
@@ -749,6 +747,6 @@
       <inertial>
          <origin xyz="7.847128413729365e-10 0.018862565434485133 0.00019573987745461708" rpy="-1.5707963267948966 -0.7853981633974787 0.0" />
-         <mass value="0.0451896335" />
-         <inertia ixx="8.98764124e-06" iyy="8.98764124e-06" izz="7.5342151e-06" ixy="2.44391272e-06" iyz="4.13205914e-08" ixz="-4.13205914e-08" />
+         <mass value="0.2245232082016773" />
+         <inertia ixx="4.46548e-05" iyy="4.46548e-05" izz="3.74335e-05" ixy="1.2142500000000001e-05" iyz="2.0530000000000002e-07" ixz="-2.0530000000000002e-07" />
       </inertial>
       <visual>
@@ -811,6 +809,6 @@
       <inertial>
          <origin xyz="0.08878055288596076 -0.03188492529312713 0.030995648486683028" rpy="1.5707963267948966 0.0 1.5707963267948966" />
-         <mass value="0.0398443972" />
-         <inertia ixx="2.81053284e-05" iyy="3.02419834e-05" izz="2.81289574e-05" ixy="-7.92075283e-07" iyz="-7.88472562e-07" ixz="-4.25483343e-08" />
+         <mass value="0.19796557769577772" />
+         <inertia ixx="0.0001396404" iyy="0.00015025630000000003" izz="0.0001397578" ixy="-3.9354000000000005e-06" iyz="-3.9175e-06" ixz="-2.114e-07" />
       </inertial>
    </link>
@@ -818,6 +816,6 @@
       <inertial>
          <origin xyz="0.08878055288596079 -0.03188492529312709 0.030995648486683187" rpy="1.5707963267948966 0.7853981633974532 1.5707963267948966" />
-         <mass value="0.0398443972" />
-         <inertia ixx="2.99657412e-05" iyy="2.83815705e-05" izz="2.81289574e-05" ixy="-1.06831742e-06" iyz="-5.8760578e-07" ixz="5.2744638e-07" />
+         <mass value="0.19796557769577772" />
+         <inertia ixx="0.00014888380000000002" iyy="0.00014101290000000002" izz="0.0001397578" ixy="-5.3079000000000005e-06" iyz="-2.9194999999999997e-06" ixz="2.6206e-06" />
       </inertial>
    </link>
@@ -825,6 +823,6 @@
       <inertial>
          <origin xyz="0.0887805528859608 -0.031884925293127184 0.030995648486683063" rpy="-1.5707963267948966 0.0 -1.5707963267948966" />
-         <mass value="0.0398443972" />
-         <inertia ixx="2.81053284e-05" iyy="3.02419834e-05" izz="2.81289574e-05" ixy="-7.92075283e-07" iyz="7.88472562e-07" ixz="4.25483343e-08" />
+         <mass value="0.19796557769577772" />
+         <inertia ixx="0.0001396404" iyy="0.00015025630000000003" izz="0.0001397578" ixy="-3.9354000000000005e-06" iyz="3.9175e-06" ixz="2.114e-07" />
       </inertial>
    </link>
@@ -832,6 +830,6 @@
       <inertial>
          <origin xyz="0.08878055288596072 -0.03188492529312713 0.030995648486683118" rpy="-1.5707963267948966 0.7853981633974585 -1.5707963267948966" />
-         <mass value="0.0398443972" />
-         <inertia ixx="2.83815705e-05" iyy="2.99657412e-05" izz="2.81289574e-05" ixy="1.06831742e-06" iyz="5.2744638e-07" ixz="5.8760578e-07" />
+         <mass value="0.19796557769577772" />
+         <inertia ixx="0.00014101290000000002" iyy="0.00014888380000000002" izz="0.0001397578" ixy="5.3079000000000005e-06" iyz="2.6206e-06" ixz="2.9194999999999997e-06" />
       </inertial>
    </link>
@@ -839,6 +837,6 @@
       <inertial>
          <origin xyz="-1.67667956555384e-05 -0.010100263506804588 -0.0033385992686390197" rpy="-1.5707963267948966 1.5568472989183801 1.5707963267948966" />
-         <mass value="0.016897885" />
-         <inertia ixx="3.27626199e-06" iyy="1.30297531e-05" izz="1.41944383e-05" ixy="-3.1784451e-07" iyz="8.45331145e-10" ixz="-1.0063466e-10" />
+         <mass value="0.08395658588476052" />
+         <inertia ixx="1.6278000000000002e-05" iyy="6.47379e-05" izz="7.05246e-05" ixy="-1.5792e-06" iyz="4.2e-09" ixz="-5e-10" />
       </inertial>
       <visual>
@@ -866,6 +864,6 @@
       <inertial>
          <origin xyz="0.0095 -0.005 0.0102" rpy="-1.5707963267948966 0.0 0.0" />
-         <mass value="0.00092261234" />
-         <inertia ixx="1.25189517e-08" iyy="1.25189517e-08" izz="2.13949287e-08" ixy="0" iyz="0" ixz="-0" />
+         <mass value="0.004583969076466208" />
+         <inertia ixx="6.22e-08" iyy="6.22e-08" izz="1.063e-07" ixy="0.0" iyz="0.0" ixz="-0.0" />
       </inertial>
       <visual>
@@ -886,6 +884,6 @@
       <inertial>
          <origin xyz="-0.0034000000000000002 0.054600389866879796 0.00940392681215343" rpy="-1.5707963267948966 -0.013949027876515308 0.0" />
-         <mass value="0.00143034466" />
-         <inertia ixx="3.31893109e-08" iyy="3.31893109e-08" izz="5.91933071e-08" ixy="0" iyz="-0" ixz="0" />
+         <mass value="0.007106620431515159" />
+         <inertia ixx="1.649e-07" iyy="1.649e-07" izz="2.941e-07" ixy="0.0" iyz="-0.0" ixz="0.0" />
       </inertial>
       <visual>
@@ -906,6 +904,6 @@
       <inertial>
          <origin xyz="0.0 0.002194420664876953 0.0" rpy="-1.5707963267948966 0.0 0.0" />
-         <mass value="0.000671356652" />
-         <inertia ixx="9.56029271e-09" iyy="9.56029271e-09" izz="1.38674562e-08" ixy="0" iyz="0" ixz="-0" />
+         <mass value="0.00333561345514696" />
+         <inertia ixx="4.75e-08" iyy="4.75e-08" izz="6.890000000000001e-08" ixy="0.0" iyz="0.0" ixz="-0.0" />
       </inertial>
       <visual>
@@ -926,6 +924,6 @@
       <inertial>
          <origin xyz="-0.0034000000000000002 0.0546003898668798 0.009403926812153412" rpy="1.5707963267948966 0.01394902787650576 1.5707963267948966" />
-         <mass value="0.00143034466" />
-         <inertia ixx="5.91933071e-08" iyy="3.31893109e-08" izz="3.31893109e-08" ixy="3.62284776e-10" iyz="-0" ixz="0" />
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