Commit message: Updated folder structure & project design

File: software/ros2_ws/src/vector_description/urdf/vector.urdf.xacro (robot description, xacro)
@@ -112,4 +112,11 @@
       <origin xyz="${lt} 0 0"/>
     </joint>
+    <!-- ToF sensor frame, x along the beam (sensor_msgs/Range on legs/${name}/tof) -->
+    <link name="${name}_tof"/>
+    <joint name="${name}_tof_joint" type="fixed">
+      <parent link="${name}_coxa_link"/>
+      <child link="${name}_tof"/>
+      <origin xyz="${g['tof']['x']} 0 ${g['tof']['z']}" rpy="0 ${g['tof']['pitch']} 0"/>
+    </joint>
   </xacro:macro>
   <xacro:leg name="L1"/>
@@ -152,8 +159,10 @@
     <xacro:leg_if name="R2"/>
     <xacro:leg_if name="R3"/>
-    <!-- leg power: command 1/0 switches the legs on/off, state is 1 once all six are active -->
+    <!-- leg power: command 1/0 switches the legs on/off, state is 1 once all six are active;
+         estop 1 sets the e-stop flag in SYNC and holds the legs off -->
     <xacro:unless value="${gazebo}">
       <gpio name="legs">
         <command_interface name="enable"/>
+        <command_interface name="estop"/>
         <state_interface name="enable"><param name="initial_value">1.0</param></state_interface>
       </gpio>

Commit message: Added GNSS, ToF sensors + obstacle mapping

File: software/ros2_ws/src/vector_description/urdf/vector.urdf.xacro (robot description, xacro)
@@ -47,4 +47,18 @@
     <child link="body_mass"/>
   </joint>
+  <!-- nose board: VL53L8CX (x along its axis) with the camera beside it; placeholder pose -->
+  <link name="nose_tof"/>
+  <joint name="nose_tof_joint" type="fixed">
+    <parent link="base_link"/>
+    <child link="nose_tof"/>
+    <origin xyz="0.12 0 0.02"/>
+  </joint>
+  <!-- GNSS antenna on the top plate (placeholder until the shell is drawn) -->
+  <link name="gnss"/>
+  <joint name="gnss_joint" type="fixed">
+    <parent link="base_link"/>
+    <child link="gnss"/>
+    <origin xyz="-0.05 0 0.08"/>
+  </joint>
   <!-- segment along +x of its own frame, mass spread along it -->
   <xacro:macro name="segment" params="name length radius m">
@@ -177,4 +191,21 @@
         <topic>imu</topic>
         <gz_frame_id>base_link</gz_frame_id>
+        <!-- yaw 0 = east, what navsat_transform expects -->
+        <imu><orientation_reference_frame><localization>ENU</localization></orientation_reference_frame></imu>
+      </sensor>
+    </gazebo>
+    <!-- GNSS: 5 Hz, 0.5 m noise (a real receiver is nearer 1.5-2.5 m, but this keeps the test short) -->
+    <gazebo reference="gnss">
+      <sensor name="gnss" type="navsat">
+        <always_on>true</always_on>
+        <update_rate>5</update_rate>
+        <topic>gnss/fix</topic>
+        <gz_frame_id>gnss</gz_frame_id>
+        <navsat>
+          <position_sensing>
+            <horizontal><noise type="gaussian"><stddev>0.5</stddev></noise></horizontal>
+            <vertical><noise type="gaussian"><stddev>1.0</stddev></noise></vertical>
+          </position_sensing>
+        </navsat>
       </sensor>
     </gazebo>

Commit message: move the leg tof to the tibia, placed from the CAD

File: software/ros2_ws/src/vector_description/urdf/vector.urdf.xacro (robot description, xacro)
@@ -129,5 +129,5 @@
     <link name="${name}_tof"/>
     <joint name="${name}_tof_joint" type="fixed">
-      <parent link="${name}_coxa_link"/>
+      <parent link="${name}_tibia_link"/>
       <child link="${name}_tof"/>
       <origin xyz="${g['tof']['x']} 0 ${g['tof']['z']}" rpy="0 ${g['tof']['pitch']} 0"/>

Commit message: Added more features
  1. Gazebo sensors
  2. black box
  3. battery time
  4. return home
  5. calibration wizard

File: software/ros2_ws/src/vector_description/urdf/vector.urdf.xacro (robot description, xacro)
@@ -54,4 +54,12 @@
     <origin xyz="0.12 0 0.02"/>
   </joint>
+  <!-- LDS01RR lidar on the top plate, its 0 deg forward once lidar_yaw is set in io_bridge
+       (placeholder height: the top plate plus the beam's ~40 mm) -->
+  <link name="lidar"/>
+  <joint name="lidar_joint" type="fixed">
+    <parent link="base_link"/>
+    <child link="lidar"/>
+    <origin xyz="0 0 0.055"/>
+  </joint>
   <!-- GNSS antenna on the top plate (placeholder until the shell is drawn) -->
   <link name="gnss"/>
@@ -133,4 +141,21 @@
       <origin xyz="${g['tof']['x']} 0 ${g['tof']['z']}" rpy="0 ${g['tof']['pitch']} 0"/>
     </joint>
+    <!-- in Gazebo, one ray along the beam (sim_tof.py makes it a Range like leg_monitor's);
+         1.3 m like the VL53L1X in short mode -->
+    <xacro:if value="${gazebo}">
+      <gazebo reference="${name}_tof">
+        <sensor name="${name}_tof" type="gpu_lidar">
+          <always_on>true</always_on>
+          <update_rate>30</update_rate>
+          <topic>legs/${name}/tof_scan</topic>
+          <gz_frame_id>${name}_tof</gz_frame_id>
+          <lidar>
+            <scan><horizontal><samples>1</samples><min_angle>0</min_angle><max_angle>0</max_angle></horizontal></scan>
+            <range><min>0.04</min><max>1.3</max></range>
+            <noise><type>gaussian</type><mean>0</mean><stddev>0.005</stddev></noise>
+          </lidar>
+        </sensor>
+      </gazebo>
+    </xacro:if>
   </xacro:macro>
   <xacro:leg name="L1"/>
@@ -195,4 +220,18 @@
       </sensor>
     </gazebo>
+    <!-- the LDS01RR: 360 points a turn at 5 turns a second, 0.15-6 m -->
+    <gazebo reference="lidar">
+      <sensor name="lidar" type="gpu_lidar">
+        <always_on>true</always_on>
+        <update_rate>5</update_rate>
+        <topic>scan</topic>
+        <gz_frame_id>lidar</gz_frame_id>
+        <lidar>
+          <scan><horizontal><samples>360</samples><min_angle>-3.14159</min_angle><max_angle>3.13414</max_angle></horizontal></scan>
+          <range><min>0.15</min><max>6.0</max></range>
+          <noise><type>gaussian</type><mean>0</mean><stddev>0.01</stddev></noise>
+        </lidar>
+      </sensor>
+    </gazebo>
     <!-- GNSS: 5 Hz, about 0.5 m of noise (a real receiver is nearer 1.5-2.5 m, but this keeps the
          test short). Gazebo applies the horizontal noise to latitude and longitude in degrees. -->
